Commit message: Squashed commit of the following:
commit 1b05ec542302a034dc62f85bd28513b43ef17223
Author: Chris Iverach-Brereton <civerachb@clearpathrobotics.com>
Date:   Wed Nov 10 09:54:43 2021 -0500

    Remove old dependencies, add the joint state controller for use inside gazebo

commit 6cef209cd4cef2212a11ff85a403b9408fbc9054
Author: Chris Iverach-Brereton <civerachb@clearpathrobotics.com>
Date:   Tue Nov 9 17:18:26 2021 -0500

    Add gazebo plugin definitions for the realsense, front & rear lidars. Move the IMU configuration into the sensors file

commit 5141445c9a09713e9a17f0501f1805c1092c4a3b
Author: Chris Iverach-Brereton <civerachb@clearpathrobotics.com>
Date:   Tue Nov 9 17:17:36 2021 -0500

    Adjust the velocity controller and friction properties to get the robot to steer better in gazebo when using the game controller. It's still a bit sluggish when turning, but better than it was

commit 8a031d0163be02efe809fb02b3ef04f5e3865ab3
Author: Chris Iverach-Brereton <civerachb@clearpathrobotics.com>
Date:   Tue Nov 9 16:07:25 2021 -0500

    Add relays so that the twist_mux output can talk to gazebo's cmd_vel input

commit cdbe72bb1704d5847f1c42f5e0459d3cfa406bda
Author: Chris Iverach-Brereton <civerachb@clearpathrobotics.com>
Date:   Tue Nov 9 13:24:32 2021 -0500

    Start progress on getting the Gazebo simulation of the new boxer to work correctly

File: boxer_description/urdf/include/sensors.urdf.xacro (robot description, xacro)
@@ -12,4 +12,62 @@
     <origin xyz="0 0 0" rpy="0 0 0" />
   </xacro:sensor_d435>
+  <!--
+    The D435 doesn't natively provide simulation data, so include the kinect plugin to make the sensor work
+    Note that the realsense on the Boxer via the Otto API only publishes the depth image, not pointcloud data
+    The gazebo kinect plugin aligns the depth data with the Z axis, with X=left and Y=up
+    ROS expects the depth data along the X axis, with Y=left and Z=up
+    This link only exists to give the gazebo plugin the correctly-oriented frame
+  -->
+  <link name="realsense_front_camera_gazebo_link" />
+  <joint name="realsense_front_camera_gazebo_joint" type="fixed">
+    <parent link="realsense_front_camera_link"/>
+    <child link="realsense_front_camera_gazebo_link"/>
+    <origin xyz="0.0 0 0" rpy="-1.5707963267948966 0 -1.5707963267948966"/>
+  </joint>
+  <gazebo reference="realsense_front_camera_link">
+    <turnGravityOff>true</turnGravityOff>
+    <sensor type="depth" name="realsense_front_camera">
+      <update_rate>30</update_rate>
+      <camera>
+        <!-- 75x65 degree FOV for the depth sensor -->
+        <horizontal_fov>1.5184351666666667</horizontal_fov>
+        <vertical_fov>1.0122901111111111</vertical_fov>
+        <image>
+          <width>640</width>
+          <height>480</height>
+          <format>RGB8</format>
+        </image>
+        <clip>
+          <!-- give the color sensor a maximum range of 50m so that the simulation renders nicely -->
+          <near>0.01</near>
+          <far>50.0</far>
+        </clip>
+      </camera>
+      <plugin name="kinect_controller" filename="libgazebo_ros_openni_kinect.so">
+        <baseline>0.2</baseline>
+        <alwaysOn>true</alwaysOn>
+        <updateRate>30</updateRate>
+        <cameraName>realsense</cameraName>
+        <imageTopicName>color/image_raw</imageTopicName>
+        <cameraInfoTopicName>color/camera_info</cameraInfoTopicName>
+        <depthImageTopicName>depth/image_rect_raw</depthImageTopicName>
+        <depthImageInfoTopicName>depth/camera_info</depthImageInfoTopicName>
+        <pointCloudTopicName>depth/color/points</pointCloudTopicName>
+        <frameName>realsense_front_camera_gazebo_link</frameName>
+        <pointCloudCutoff>0.105</pointCloudCutoff>
+        <pointCloudCutoffMax>8.0</pointCloudCutoffMax>
+        <distortionK1>0.00000001</distortionK1>
+        <distortionK2>0.00000001</distortionK2>
+        <distortionK3>0.00000001</distortionK3>
+        <distortionT1>0.00000001</distortionT1>
+        <distortionT2>0.00000001</distortionT2>
+        <CxPrime>0</CxPrime>
+        <Cx>0</Cx>
+        <Cy>0</Cy>
+        <focalLength>0</focalLength>
+        <hackBaseline>0</hackBaseline>
+      </plugin>
+    </sensor>
+  </gazebo>
   <!-- Front safety sensor -->
   <link name="front_laser">
@@ -27,6 +85,38 @@
     <origin xyz="0.3062 0 0.1614" rpy="0 0 0" />
   </joint>
+  <gazebo reference="front_laser">
+    <turnGravityOff>true</turnGravityOff>
+    <sensor type="ray" name="front_laser">
+      <pose>0 0 0 0 0 0</pose>
+      <visualize>false</visualize>
+      <update_rate>33</update_rate>
+      <ray>
+        <scan>
+          <horizontal>
+            <samples>720</samples>
+            <resolution>1</resolution>
+            <min_angle>-2.35619449019</min_angle>
+            <max_angle>2.35619449019</max_angle>
+          </horizontal>
+        </scan>
+        <range>
+          <min>0.5</min>
+          <max>20</max>
+          <resolution>0.01</resolution>
+        </range>
+        <noise>
+          <type>gaussian</type>
+          <mean>0.0</mean>
+          <stddev>0.001</stddev>
+        </noise>
+      </ray>
+      <plugin name="gazebo_ros_laser" filename="libgazebo_ros_laser.so">
+        <topicName>front/scan</topicName>
+        <frameName>front_laser</frameName>
+        <robotNamespace>/</robotNamespace>
+      </plugin>
+    </sensor>
+  </gazebo>
   <!-- Internal rear safety laser -->
-  <!-- TODO: enable a gazebo plugin for this sensor -->
   <link name="rear_sensor">
     <visual>
@@ -43,4 +133,38 @@
     <origin xyz="-0.3404 0.0241 0.0779" rpy="0 -0.0698131700798 ${pi}" />
   </joint>
+  <!-- TODO look up the actual specs for this sensor; range, FoV, samples is a complete guess right now -->
+  <gazebo reference="rear_sensor">
+    <turnGravityOff>true</turnGravityOff>
+    <sensor type="ray" name="rear_laser">
+      <pose>0 0 0 0 0 0</pose>
+      <visualize>false</visualize>
+      <update_rate>33</update_rate>
+      <ray>
+        <scan>
+          <horizontal>
+            <samples>90</samples>
+            <resolution>1</resolution>
+            <min_angle>0.785398163397</min_angle>
+            <max_angle>-0.785398163397</max_angle>
+          </horizontal>
+        </scan>
+        <range>
+          <min>0.1</min>
+          <max>5</max>
+          <resolution>0.01</resolution>
+        </range>
+        <noise>
+          <type>gaussian</type>
+          <mean>0.0</mean>
+          <stddev>0.001</stddev>
+        </noise>
+      </ray>
+      <plugin name="gazebo_ros_laser" filename="libgazebo_ros_laser.so">
+        <topicName>rear/scan</topicName>
+        <frameName>rear_sensor</frameName>
+        <robotNamespace>/</robotNamespace>
+      </plugin>
+    </sensor>
+  </gazebo>
   <!-- Cart sensor -->
   <link name="cart_sensor"/>
@@ -57,3 +181,17 @@
     <origin rpy="0 0 -0.78539816339744828" xyz="0.191959 -0.086412 0.18455965360"/>
   </joint>
+  <gazebo>
+    <plugin name="imu_controller" filename="libhector_gazebo_ros_imu.so">
+      <robotNamespace>/</robotNamespace>
+      <updateRate>50.0</updateRate>
+      <bodyName>imu_link</bodyName>
+      <topicName>/imu/module0/data</topicName>
+      <accelDrift>0.005 0.005 0.005</accelDrift>
+      <accelGaussianNoise>0.005 0.005 0.005</accelGaussianNoise>
+      <rateDrift>0.005 0.005 0.005 </rateDrift>
+      <rateGaussianNoise>0.005 0.005 0.005 </rateGaussianNoise>
+      <headingDrift>0.005</headingDrift>
+      <headingGaussianNoise>0.005</headingGaussianNoise>
+    </plugin>
+  </gazebo>
 </robot>

File: boxer_description/urdf/include/wheels_and_casters.urdf.xacro (robot description, xacro)
@@ -37,13 +37,13 @@
     </joint>
     <gazebo reference="${name}_link">
-      <material>Gazebo/Black</material>
+      <material>Gazebo/DarkGrey</material>
       <selfCollide>false</selfCollide>
-      <mu1 value="0.0"/>
-      <mu2 value="0.0"/>
-      <slip1 value="1.0" />
-      <slip2 value="1.0" />
-      <kp value="10000000.0" />
-      <kd value="1" />
-      <fdir1 value="1 0 0"/>
+      <!-- For castors, we need high PID values to avoid slippage -->
+      <kp>100000000.0</kp>
+      <kd>10000.0</kd>
+      <!-- Castors will slide freely to allow turning -->
+      <mu1>0</mu1>
+      <mu2>0</mu2>
+      <minDepth>0.0</minDepth>
     </gazebo>
   </xacro:macro>
@@ -76,12 +76,23 @@
       <dynamics damping="1.0" />
     </joint>
+    <transmission name="${name}_transmission">
+      <type>transmission_interface/SimpleTransmission</type>
+      <joint name="${name}_joint">
+        <hardwareInterface>hardware_interface/VelocityJointInterface</hardwareInterface>
+      </joint>
+      <actuator name="${name}_actuator">
+        <mechanicalReduction>1</mechanicalReduction>
+      </actuator>
+    </transmission>
     <gazebo reference="${name}_link">
       <material>Gazebo/Black</material>
       <selfCollide>false</selfCollide>
-      <mu1 value="0.5"/>
-      <mu2 value="0.5"/>
-      <kp value="10000000.0" />
-      <kd value="1" />
-      <fdir1 value="1 0 0"/>
+      <!-- For wheels, we need high PID values to avoid slippage -->
+      <kp value="100000000.0" />
+      <kd value="10000.0" />
+      <!-- Wheels have friction to prevent slippage -->
+      <mu1 value="0.1"/>
+      <mu2 value="0.1"/>
+      <minDepth>0.0</minDepth>
     </gazebo>
   </xacro:macro>
@@ -98,21 +109,3 @@
     <origin xyz="0.2436 0.1503 0.0526" rpy="0 0 0" />
   </xacro:drive_wheel>
-  <transmission name="wheel_left_transmission">
-    <type>transmission_interface/SimpleTransmission</type>
-    <joint name="wheel_left_joint">
-      <hardwareInterface>hardware_interface/VelocityJointInterface</hardwareInterface>
-    </joint>
-    <actuator name="wheel_left_actuator">
-      <mechanicalReduction>1</mechanicalReduction>
-    </actuator>
-  </transmission>
-  <transmission name="wheel_right_transmission">
-    <type>transmission_interface/SimpleTransmission</type>
-    <joint name="wheel_right_joint">
-      <hardwareInterface>hardware_interface/VelocityJointInterface</hardwareInterface>
-    </joint>
-    <actuator name="wheel_right_actuator">
-      <mechanicalReduction>1</mechanicalReduction>
-    </actuator>
-  </transmission>
 </robot>

Commit message: Add gazebo materials for the realsense and lidars so they don't render in pure-white inside the simulation

File: boxer_description/urdf/include/sensors.urdf.xacro (robot description, xacro)
@@ -26,4 +26,5 @@
   </joint>
   <gazebo reference="realsense_front_camera_link">
+    <material>Gazebo/Black</material>
     <turnGravityOff>true</turnGravityOff>
     <sensor type="depth" name="realsense_front_camera">
@@ -86,4 +87,5 @@
   </joint>
   <gazebo reference="front_laser">
+    <material>Gazebo/Black</material>
     <turnGravityOff>true</turnGravityOff>
     <sensor type="ray" name="front_laser">
@@ -135,4 +137,5 @@
   <!-- TODO look up the actual specs for this sensor; range, FoV, samples is a complete guess right now -->
   <gazebo reference="rear_sensor">
+    <material>Gazebo/Black</material>
     <turnGravityOff>true</turnGravityOff>
     <sensor type="ray" name="rear_laser">
