Commit message: Add support for the ECX-1000 series vecow backpack

File: boxer_description/urdf/boxer.urdf.xacro (robot description, xacro)
@@ -76,4 +76,11 @@
       </xacro:vecow_evs2000>
     </xacro:if>
+    <!-- Alternate Vecow: ECX-1000 series -->
+    <xacro:if value="${pc_model == 'ecx-1000'}">
+      <xacro:include filename="$(find boxer_description)/urdf/include/vecow_ecx1000.urdf.xacro" />
+      <xacro:vecow_ecx1000 prefix="vecow" parent="top_plate_link">
+        <origin xyz="0.0575 0 0" rpy="0 0 0" />
+      </xacro:vecow_ecx1000>
+    </xacro:if>
     <!-- Commercial mini-ITX motherboard with a mini case -->
     <xacro:if value="${pc_model == 'mini-itx'}">

Commit message: Add ECX-2000 URDF for backpack computer; removed unsupported ECX-1000

File: boxer_description/urdf/boxer.urdf.xacro (robot description, xacro)
@@ -76,10 +76,10 @@
       </xacro:vecow_evs2000>
     </xacro:if>
-    <!-- Alternate Vecow: ECX-1000 series -->
-    <xacro:if value="${pc_model == 'ecx-1000'}">
-      <xacro:include filename="$(find boxer_description)/urdf/include/vecow_ecx1000.urdf.xacro" />
-      <xacro:vecow_ecx1000 prefix="vecow" parent="top_plate_link">
-        <origin xyz="0.0575 0 0" rpy="0 0 0" />
-      </xacro:vecow_ecx1000>
+    <!-- Alternate Vecow: ECX-2000 series -->
+    <xacro:if value="${pc_model == 'ecx-2000'}">
+      <xacro:include filename="$(find boxer_description)/urdf/include/vecow_ecx2000.urdf.xacro" />
+      <xacro:vecow_ecx2000 prefix="vecow" parent="top_plate_link">
+        <origin xyz="0.0575 0 0" rpy="0 0 1.57" />
+      </xacro:vecow_ecx2000>
     </xacro:if>
     <!-- Commercial mini-ITX motherboard with a mini case -->

Commit message: Add BOXER_PC_XYZ and BOXER_PC_RPY envars to support relocating backpack computer in URDF

File: boxer_description/urdf/boxer.urdf.xacro (robot description, xacro)
@@ -73,5 +73,5 @@
       <xacro:include filename="$(find boxer_description)/urdf/include/vecow_evs2000.urdf.xacro" />
       <xacro:vecow_evs2000 prefix="vecow" parent="top_plate_link">
-        <origin xyz="0.0575 0 0" rpy="0 0 0" />
+        <origin xyz="$(optenv BOXER_PC_XYZ 0.0575 0 0)" rpy="$(optenv BOXER_PC_RPY 0 0 0)" />
       </xacro:vecow_evs2000>
     </xacro:if>
@@ -80,5 +80,5 @@
       <xacro:include filename="$(find boxer_description)/urdf/include/vecow_ecx2000.urdf.xacro" />
       <xacro:vecow_ecx2000 prefix="vecow" parent="top_plate_link">
-        <origin xyz="0.0575 0 0" rpy="0 0 1.57" />
+        <origin xyz="$(optenv BOXER_PC_XYZ 0.0575 0 0)" rpy="$(optenv BOXER_PC_RPY 0 0 1.57)" />
       </xacro:vecow_ecx2000>
     </xacro:if>
@@ -87,5 +87,5 @@
       <xacro:include filename="$(find boxer_description)/urdf/include/mini_itx.urdf.xacro" />
       <xacro:mini_itx prefix="pc" parent="top_plate_link">
-        <origin xyz="0.0575 0 0" rpy="0 0 0" />
+        <origin xyz="$(optenv BOXER_PC_XYZ 0.0575 0 0)" rpy="$(optenv BOXER_PC_RPY 0 0 0)" />
       </xacro:mini_itx>
     </xacro:if>
